File: mix2.kicad_sch (KiCad schematic)
At the start: 39 parts, among them J1 Conn_02x05_Odd_Even, J2 in0, J3 in1, J4 in2, J5 in3, J6 out, U1 TL072

Commit message: fix bom issues
Parts:
- C3: value C -> 100n
- H10: value lvl0 -> lvl 1
- H11: value lvl1 -> lvl 2
- H12: value lvl2 -> lvl 3
- H13: value lvl3 -> lvl 4
- U1: PartNum (none) -> 595-TL072CDR; Vendor (none) -> Mouser
Other:
- moved on the sheet: C3
Changed lines of the file:
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@@
 	(wire
 		(pts
-			(xy 215.9 149.86) (xy 219.71 149.86)
+			(xy 213.36 149.86) (xy 219.71 149.86)
 		)
 		(stroke
@@
 	(wire
 		(pts
-			(xy 215.9 134.62) (xy 215.9 138.43)
+			(xy 213.36 134.62) (xy 213.36 138.43)
 		)
 		(stroke
@@
 	(wire
 		(pts
-			(xy 215.9 146.05) (xy 215.9 149.86)
+			(xy 213.36 146.05) (xy 213.36 149.86)
 		)
 		(stroke
@@
 	(wire
 		(pts
-			(xy 219.71 134.62) (xy 215.9 134.62)
+			(xy 219.71 134.62) (xy 213.36 134.62)
 		)
 		(stroke
@@
 	(symbol
 		(lib_id "Device:C")
-		(at 215.9 142.24 0)
+		(at 213.36 142.24 0)
 		(unit 1)
 		(body_style 1)
@@
 		(fields_autoplaced yes)
 		(property "Reference" "C3"
-			(at 219.71 140.9699 0)
+			(at 217.17 140.9699 0)
 			(show_name no)
 			(do_not_autoplace no)
@@
 			)
 		)
-		(property "Value" "C"
-			(at 219.71 143.5099 0)
+		(property "Value" "100n"
+			(at 217.17 143.5099 0)
 			(show_name no)
 			(do_not_autoplace no)
@@
 		)
 		(property "Footprint" "Capacitor_SMD:C_0805_2012Metric"
-			(at 216.8652 146.05 0)
+			(at 214.3252 146.05 0)
 			(hide yes)
 			(show_name no)
@@
 		)
 		(property "Datasheet" ""
-			(at 215.9 142.24 0)
+			(at 213.36 142.24 0)
 			(hide yes)
 			(show_name no)
@@
 		)
 		(property "Description" "Unpolarized capacitor"
-			(at 215.9 142.24 0)
+			(at 213.36 142.24 0)
 			(hide yes)
 			(show_name no)
@@
 			)
 		)
-		(property "Value" "lvl3"
+		(property "Value" "lvl 4"
 			(at 60.96 193.0399 0)
 			(show_name no)
@@
 			)
 		)
-		(property "Value" "lvl1"
+		(property "Value" "lvl 2"
 			(at 60.96 177.7999 0)
 			(show_name no)
@@
 			)
 		)
+		(property "Vendor" "Mouser"
+			(at 227.33 142.24 0)
+			(hide yes)
+			(show_name no)
+			(do_not_autoplace no)
+			(effects
+				(font
+					(size 1.27 1.27)
+				)
+			)
+		)
+		(property "PartNum" "595-TL072CDR"
+			(at 227.33 142.24 0)
+			(hide yes)
+			(show_name no)
+			(do_not_autoplace no)
+			(effects
+				(font
+					(size 1.27 1.27)
+				)
+			)
+		)
 		(pin "3"
 		)
@@
 			)
 		)
-		(property "Value" "lvl0"
+		(property "Value" "lvl 1"
 			(at 60.96 170.1799 0)
 			(show_name no)
@@
 			)
 		)
+		(property "Vendor" "Mouser"
+			(at 90.17 50.8 0)
+			(hide yes)
+			(show_name no)
+			(do_not_autoplace no)
+			(effects
+				(font
+					(size 1.27 1.27)
+				)
+			)
+		)
+		(property "PartNum" "595-TL072CDR"
+			(at 90.17 50.8 0)
+			(hide yes)
+			(show_name no)
+			(do_not_autoplace no)
+			(effects
+				(font
+					(size 1.27 1.27)
+				)
+			)
+		)
 		(pin "3"
 		)
@@
 			)
 		)
+		(property "Vendor" "Mouser"
+			(at 113.03 53.34 0)
+			(hide yes)
+			(show_name no)
+			(do_not_autoplace no)
+			(effects
+				(font
+					(size 1.27 1.27)
+				)
+			)
+		)
+		(property "PartNum" "595-TL072CDR"
+			(at 113.03 53.34 0)
+			(hide yes)
+			(show_name no)
+			(do_not_autoplace no)
+			(effects
+				(font
+					(size 1.27 1.27)
+				)
+			)
+		)
 		(pin "3"
 		)
@@
 			)
 		)
-		(property "Value" "lvl2"
+		(property "Value" "lvl 3"
 			(at 60.96 185.4199 0)
 			(show_name no)
