File: mix2.kicad_pcb (KiCad board)
At the start: 2 copper layers, 30 x 241.5 mm, 39 parts, among them J1 Conn_02x05_Odd_Even, J2 in0, J3 in1, J4 in2, J5 in3, J6 out, U1 TL072

Commit message: fix bom issues
Parts:
- C3: value C -> 100n
Changed lines of the file:
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@@
 			)
 		)
+		(property "Vendor" "Mouser"
+			(at 0 0 270)
+			(unlocked yes)
+			(layer "F.Fab")
+			(hide yes)
+			(effects
+				(font
+					(size 1 1)
+					(thickness 0.15)
+				)
+			)
+		)
+		(property "PartNum" "595-TL072CDR"
+			(at 0 0 270)
+			(unlocked yes)
+			(layer "F.Fab")
+			(hide yes)
+			(effects
+				(font
+					(size 1 1)
+					(thickness 0.15)
+				)
+			)
+		)
 		(property ki_fp_filters "SOIC*3.9x4.9mm*P1.27mm* DIP*W7.62mm* TO*99* OnSemi*Micro8* TSSOP*3x3mm*P0.65mm* TSSOP*4.4x3mm*P0.65mm* MSOP*3x3mm*P0.65mm* SSOP*3.9x4.9mm*P0.635mm* LFCSP*2x2mm*P0.5mm* *SIP* SOIC*5.3x6.2mm*P1.27mm*")
 		(sheetname "/")
@@
 			)
 		)
-		(property "Value" "C"
+		(property "Value" "100n"
 			(at 0 1.68 90)
 			(layer "F.Fab")

Commit message: fix alignment for manu
Parts:
- moved J1 4.70 mm to (44.6, 83.5)
- moved C2 4.70 mm to (50.0, 96.5)
- moved C3 4.70 mm to (54.3, 86.1)
- moved J2 4.70 mm to (61.3, 47.1)
- moved J3 4.70 mm to (61.3, 73.1)
- moved J4 4.70 mm to (61.3, 99.1)
- moved J5 4.70 mm to (61.3, 125.1)
- moved J6 4.70 mm to (61.3, 28.1)
- moved R10 4.70 mm to (65.3, 83.1)
- moved R3 4.70 mm to (58.3, 65.1)
- moved R4 4.70 mm to (56.3, 80.1)
- moved R5 4.70 mm to (56.3, 92.1)
- moved R6 4.70 mm to (58.3, 107.1)
- moved R7 4.70 mm to (61.3, 80.1)
- moved R8 4.70 mm to (61.3, 92.1)
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Other:
- board size 30 x 241.5 mm -> 30 x 241 mm
